File: PCB/eagle cad/lion/lion.sch (EAGLE design)
At the start: 16 parts, among them IC1 PIC18F4550_40

Commit message: PCB updated
Parts:
- added C4: 22uf, resistor:CPOL-USE2,5-6E
- added JACK9V: 9VJACK, leonino:9VJACK
- added JP1: (no value), jumper:JP2E
- added LED1: (no value), led:LEDLD260
- added R2: 1k, resistor:R-EU_0204/7
- added U$11: LM7805C, leonino:LM7805C
- added U$12: DUBOX2, leonino:DUBOX2
- C1, C2: value 18pF -> 18pf; device resistor:C-EU025-025X050 -> resistor:C-EU050-025X075
- C3: value 220nF -> 220nf; device resistor:C-EU025-025X050 -> resistor:C-EU050-025X075
- R1: device resistor:R-EU_0204/5 -> resistor:R-EU_0204/7
Connections:
- removed net N$9: IC1.VDD, R1.2
- new net +5V: JP1.1, U$1.VCC
- new net GND: BUTTON1.P12, C1.2, C2.2, C3.2, C4.-, IC1.VSS, JACK9V.GND, R2.1, U$1.GND, U$11.GND, U$12.P1
- new net N$41: JP1.3, U$11.VCC
- new net N$43: LED1.C, R2.2
- net N$1: now also IC1.RA4/T0CKI/CIOUT/RCV, LED1.A; no longer U$1.VCC
- net N$3: now also IC1.RC5/D+/VP
- net N$30: now also C4.+, JP1.2, R1.2
- net N$6: now also JACK9V.VCC, U$11.INPUT, U$12.P2; no longer BUTTON1.P12, C1.2, C2.2, C3.2, IC1.VSS, U$1.GND
- net N$8: now also IC1.RC4/D-/VM
Other:
- moved on the sheet: R1
